File: ax5043.kicad_sch (KiCad schematic)
At the start: 0 parts

Commit message: Lots of work on the documentation
Signed-off-by: Corey Minyard <corey@minyard.net>
Other:
- sheet RX_1_ax5044 renamed RX_1_ax5043
- added sheet RX_2_ax5043 (RX_2_ax5043.kicad_sch)
- added sheet RX_3_ax5043 (RX_3_ax5043.kicad_sch)
- added sheet RX_4_ax5043 (RX_4_ax5043.kicad_sch)
- added sheet TX_ax5043 (TX_ax5043.kicad_sch)
- note removed: "200"
Changed lines of the file:
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@@
 	(generator_version "9.0")
 	(paper "A4")
-	(text "200"
-		(exclude_from_sim no)
-		(at 34.29 45.72 0)
-		(effects
-			(font
-				(size 1.524 1.524)
-			)
-			(justify left bottom)
+	(sheet
+		(at 105.41 31.75)
+		(size 52.07 15.24)
+		(exclude_from_sim no)
+		(in_bom yes)
+		(on_board yes)
+		(dnp no)
+		(fields_autoplaced yes)
+		(stroke
+			(width 0.1524)
+			(type solid)
+		)
+		(fill
+			(color 0 0 0 0.0000)
+		)
+		(property "Sheetname" "TX_ax5043"
+			(at 105.41 31.0384 0)
+			(effects
+				(font
+					(size 1.27 1.27)
+				)
+				(justify left bottom)
+			)
+		)
+		(property "Sheetfile" "TX_ax5043.kicad_sch"
+			(at 105.41 47.5746 0)
+			(effects
+				(font
+					(size 1.27 1.27)
+				)
+				(justify left top)
+			)
+		)
+		(instances
+			(project "PacSat_AFSK"
+				(path "/cc9f42d2-6985-41ac-acab-5ab7b01c5b38/d9a83ee4-3280-49b9-88b8-54d26cbd8ed1"
+					(page "11")
+				)
+			)
+		)
+	)
+	(sheet
+		(at 33.02 54.61)
+		(size 52.07 15.24)
+		(exclude_from_sim no)
+		(in_bom yes)
+		(on_board yes)
+		(dnp no)
+		(fields_autoplaced yes)
+		(stroke
+			(width 0.1524)
+			(type solid)
+		)
+		(fill
+			(color 0 0 0 0.0000)
+		)
+		(property "Sheetname" "RX_2_ax5043"
+			(at 33.02 53.8984 0)
+			(effects
+				(font
+					(size 1.27 1.27)
+				)
+				(justify left bottom)
+			)
+		)
+		(property "Sheetfile" "RX_2_ax5043.kicad_sch"
+			(at 33.02 70.4346 0)
+			(effects
+				(font
+					(size 1.27 1.27)
+				)
+				(justify left top)
+			)
+		)
+		(instances
+			(project "PacSat_AFSK"
+				(path "/cc9f42d2-6985-41ac-acab-5ab7b01c5b38/d9a83ee4-3280-49b9-88b8-54d26cbd8ed1"
+					(page "8")
+				)
+			)
+		)
+	)
+	(sheet
+		(at 33.02 77.47)
+		(size 52.07 16.51)
+		(exclude_from_sim no)
+		(in_bom yes)
+		(on_board yes)
+		(dnp no)
+		(fields_autoplaced yes)
+		(stroke
+			(width 0.1524)
+			(type solid)
+		)
+		(fill
+			(color 0 0 0 0.0000)
+		)
+		(property "Sheetname" "RX_3_ax5043"
+			(at 33.02 76.7584 0)
+			(effects
+				(font
+					(size 1.27 1.27)
+				)
+				(justify left bottom)
+			)
+		)
+		(property "Sheetfile" "RX_3_ax5043.kicad_sch"
+			(at 33.02 94.5646 0)
+			(effects
+				(font
+					(size 1.27 1.27)
+				)
+				(justify left top)
+			)
+		)
+		(instances
+			(project "PacSat_AFSK"
+				(path "/cc9f42d2-6985-41ac-acab-5ab7b01c5b38/d9a83ee4-3280-49b9-88b8-54d26cbd8ed1"
+					(page "9")
+				)
+			)
+		)
+	)
+	(sheet
+		(at 33.02 102.87)
+		(size 52.07 17.78)
+		(exclude_from_sim no)
+		(in_bom yes)
+		(on_board yes)
+		(dnp no)
+		(fields_autoplaced yes)
+		(stroke
+			(width 0.1524)
+			(type solid)
+		)
+		(fill
+			(color 0 0 0 0.0000)
+		)
+		(property "Sheetname" "RX_4_ax5043"
+			(at 33.02 102.1584 0)
+			(effects
+				(font
+					(size 1.27 1.27)
+				)
+				(justify left bottom)
+			)
+		)
+		(property "Sheetfile" "RX_4_ax5043.kicad_sch"
+			(at 33.02 121.2346 0)
+			(effects
+				(font
+					(size 1.27 1.27)
+				)
+				(justify left top)
+			)
+		)
+		(instances
+			(project "PacSat_AFSK"
+				(path "/cc9f42d2-6985-41ac-acab-5ab7b01c5b38/d9a83ee4-3280-49b9-88b8-54d26cbd8ed1"
+					(page "10")
+				)
+			)
 		)
 	)
@@
 			(color 0 0 0 0.0000)
 		)
-		(property "Sheetname" "RX_1_ax5044"
+		(property "Sheetname" "RX_1_ax5043"
 			(at 33.02 30.9114 0)
 			(effects
@@
 		)
 		(instances
-			(project "PacSat_AFSK"
-				(path "/cc9f42d2-6985-41ac-acab-5ab7b01c5b38/08b601c8-ef5c-4c4a-8b80-34005eff379c"
-					(page "3")
-				)
-			)
+			(project ""
+				(path "/d9a83ee4-3280-49b9-88b8-54d26cbd8ed1"
+					(page "")
+				)
+			)
+			(project "PacSat_AFSK"
+				(path "/cc9f42d2-6985-41ac-acab-5ab7b01c5b38/d9a83ee4-3280-49b9-88b8-54d26cbd8ed1"
+					(page "7")
+				)
+			)
