File: Power_Amp.kicad_sch (KiCad schematic)
At the start: 27 parts, among them J10 2118718-2, J11 Molex 73251-1153, P13 CONUFL001-SMD-T, U27 TQP7M9106, U28 ADL5501AKSZ-R2, U29 ADL5501AKSZ-R2

Commit message: More work on various things
Signed-off-by: Corey Minyard <corey@minyard.net>
Parts:
- added H20, H21: Wire_Hole, PacSatDev_misc:Wire_Hole, symbol PACSAT_DEV_misc:CUBESAT_MOUNT_HOLE_1
Connections:
- net GND: now also H20.1, H21.1
Changed lines of the file:
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@@
 	)
 	(junction
+		(at 267.97 114.3)
+		(diameter 0)
+		(color 0 0 0 0)
+	)
+	(junction
 		(at 147.32 142.24)
 		(diameter 0)
@@
 	(wire
 		(pts
+			(xy 252.73 114.3) (xy 267.97 114.3)
+		)
+		(stroke
+			(width 0)
+			(type default)
+		)
+	)
+	(wire
+		(pts
 			(xy 83.82 160.02) (xy 83.82 162.56)
 		)
@@
 	(wire
 		(pts
+			(xy 252.73 105.41) (xy 267.97 105.41)
+		)
+		(stroke
+			(width 0)
+			(type default)
+		)
+	)
+	(wire
+		(pts
 			(xy 153.67 217.17) (xy 163.83 217.17)
 		)
@@
 	(wire
 		(pts
+			(xy 267.97 114.3) (xy 267.97 116.84)
+		)
+		(stroke
+			(width 0)
+			(type default)
+		)
+	)
+	(wire
+		(pts
 			(xy 398.78 100.33) (xy 405.13 100.33)
 		)
@@
 	(wire
 		(pts
+			(xy 267.97 105.41) (xy 267.97 114.3)
+		)
+		(stroke
+			(width 0)
+			(type default)
+		)
+	)
+	(wire
+		(pts
 			(xy 405.13 100.33) (xy 405.13 74.93)
 		)
@@
 	)
 	(symbol
+		(lib_id "PACSAT_DEV_misc:CUBESAT_MOUNT_HOLE_1")
+		(at 250.19 105.41 0)
+		(unit 1)
+		(exclude_from_sim no)
+		(in_bom yes)
+		(on_board yes)
+		(dnp no)
+		(property "Reference" "H20"
+			(at 250.9774 99.3902 0)
+			(effects
+				(font
+					(size 1.524 1.524)
+				)
+			)
+		)
+		(property "Value" "Wire_Hole"
+			(at 250.9774 102.0826 0)
+			(effects
+				(font
+					(size 1.524 1.524)
+				)
+			)
+		)
+		(property "Footprint" "PacSatDev_misc:Wire_Hole"
+			(at 250.19 105.41 0)
+			(effects
+				(font
+					(size 1.524 1.524)
+				)
+				(hide yes)
+			)
+		)
+		(property "Datasheet" ""
+			(at 250.19 105.41 0)
+			(effects
+				(font
+					(size 1.524 1.524)
+				)
+				(hide yes)
+			)
+		)
+		(property "Description" ""
+			(at 250.19 105.41 0)
+			(effects
+				(font
+					(size 1.27 1.27)
+				)
+			)
+		)
+		(pin "1"
+		)
+		(instances
+			(project "PacSat_AFSK"
+				(path "/cc9f42d2-6985-41ac-acab-5ab7b01c5b38/b85b88c3-87c5-49e2-804e-0759552ace3d"
+					(reference "H20")
+					(unit 1)
+				)
+			)
+		)
+	)
+	(symbol
 		(lib_id "power:GND")
 		(at 163.83 228.6 0)
@@
 	)
 	(symbol
+		(lib_id "power:GND")
+		(at 267.97 116.84 0)
+		(unit 1)
+		(exclude_from_sim no)
+		(in_bom yes)
+		(on_board yes)
+		(dnp no)
+		(property "Reference" "#PWR0257"
+			(at 267.97 123.19 0)
+			(effects
+				(font
+					(size 1.27 1.27)
+				)
+				(hide yes)
+			)
+		)
+		(property "Value" "GND"
+			(at 268.097 121.2342 0)
+			(effects
+				(font
+					(size 1.27 1.27)
+				)
+			)
+		)
+		(property "Footprint" ""
+			(at 267.97 116.84 0)
+			(effects
+				(font
+					(size 1.27 1.27)
+				)
+				(hide yes)
+			)
+		)
+		(property "Datasheet" ""
+			(at 267.97 116.84 0)
+			(effects
+				(font
+					(size 1.27 1.27)
+				)
+				(hide yes)
+			)
+		)
+		(property "Description" ""
+			(at 267.97 116.84 0)
+			(effects
+				(font
+					(size 1.27 1.27)
+				)
+			)
+		)
+		(pin "1"
+		)
+		(instances
+			(project "PacSat_AFSK"
+				(path "/cc9f42d2-6985-41ac-acab-5ab7b01c5b38/b85b88c3-87c5-49e2-804e-0759552ace3d"
+					(reference "#PWR0257")
+					(unit 1)
+				)
+			)
+		)
+	)
+	(symbol
 		(lib_id "PACSAT_DEV_misc:LFCG-490+")
 		(at 302.26 160.02 0)
@@
 					(unit 1)
 				)
+			)
+		)
+	)
+	(symbol
+		(lib_id "PACSAT_DEV_misc:CUBESAT_MOUNT_HOLE_1")
+		(at 250.19 114.3 0)
+		(unit 1)
+		(exclude_from_sim no)
+		(in_bom yes)
+		(on_board yes)
+		(dnp no)
+		(property "Reference" "H21"
+			(at 250.9774 108.2802 0)
+			(effects
+				(font
+					(size 1.524 1.524)
+				)
+			)
+		)
+		(property "Value" "Wire_Hole"
+			(at 250.9774 110.9726 0)
+			(effects
+				(font
+					(size 1.524 1.524)
+				)
+			)
+		)
+		(property "Footprint" "PacSatDev_misc:Wire_Hole"
+			(at 250.19 114.3 0)
+			(effects
+				(font
+					(size 1.524 1.524)
+				)
+				(hide yes)
+			)
+		)
+		(property "Datasheet" ""
+			(at 250.19 114.3 0)
+			(effects
+				(font
+					(size 1.524 1.524)
+				)
+				(hide yes)
+			)
+		)
+		(property "Description" ""
+			(at 250.19 114.3 0)
+			(effects
+				(font
+					(size 1.27 1.27)
+				)
+			)
+		)
+		(pin "1"
+		)
+		(instances
+			(project "PacSat_AFSK"
+				(path "/cc9f42d2-6985-41ac-acab-5ab7b01c5b38/b85b88c3-87c5-49e2-804e-0759552ace3d"
+					(reference "H21")
+					(unit 1)
+				)

Commit message: More wokr on the PA
Fix some values on the PA and rearrange a bit to get the inductors
away from each other.

Signed-off-by: Corey Minyard <corey@minyard.net>
Parts:
- L37: value 18n -> 36n Q>40 I>1A; footprint Inductor_SMD:L_0805_2012Metric_Pad1.05x1.20mm_HandSolder -> Inductor_SMD:L_0603_1608Metric_Pad1.05x0.95mm_HandSolder
- R78: value 240 -> 280
Connections:
- net SSPA_VCC: now also L36.2; no longer R79.1
- net at L36.1: now also R79.1; no longer U27.18 (IREF)
- net at R79.2: now also U27.18 (IREF); no longer L36.2
Other:
- moved on the sheet: L36, R79
Changed lines of the file:
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@@
 	(symbol
 		(lib_id "Device:L")
-		(at 160.02 142.24 180)
+		(at 160.02 121.92 180)
 		(unit 1)
 		(exclude_from_sim no)
@@
 		(dnp no)
 		(property "Reference" "L36"
-			(at 161.798 142.24 90)
+			(at 161.798 121.92 90)
 			(effects
 				(font
@@
 		)
 		(property "Value" "68n"
-			(at 157.226 141.478 90)
+			(at 157.226 121.158 90)
 			(effects
 				(font
@@
 		)
 		(property "Footprint" "Inductor_SMD:L_0603_1608Metric_Pad1.05x0.95mm_HandSolder"
-			(at 160.02 142.24 0)
+			(at 160.02 121.92 0)
 			(effects
 				(font
@@
 		)
 		(property "Datasheet" "~"
-			(at 160.02 142.24 0)
-			(effects
-				(font
-					(size 1.27 1.27)
-				)
-				(hide yes)
-			)
-		)
-		(property "Description" ""
-			(at 160.02 142.24 0)
+			(at 160.02 121.92 0)
+			(effects
+				(font
+					(size 1.27 1.27)
+				)
+				(hide yes)
+			)
+		)
+		(property "Description" ""
+			(at 160.02 121.92 0)
 			(effects
 				(font
@@
 			)
 		)
-		(property "Value" "18n"
+		(property "Value" "36n Q>40 I>1A"
 			(at 191.77 140.716 90)
 			(effects
@@
 			)
 		)
-		(property "Footprint" "Inductor_SMD:L_0805_2012Metric_Pad1.05x1.20mm_HandSolder"
+		(property "Footprint" "Inductor_SMD:L_0603_1608Metric_Pad1.05x0.95mm_HandSolder"
 			(at 194.31 140.97 0)
 			(effects
@@
 			)
 		)
-		(property "Value" "240"
+		(property "Value" "280"
 			(at 84.836 109.728 90)
 			(effects
@@
 	(symbol
 		(lib_id "Device:R")
-		(at 160.02 121.92 0)
+		(at 160.02 142.24 0)
 		(unit 1)
 		(exclude_from_sim no)
@@
 		(dnp no)
 		(property "Reference" "R79"
-			(at 157.48 124.46 90)
+			(at 157.48 144.78 90)
 			(effects
 				(font
@@
 		)
 		(property "Value" "240"
-			(at 162.306 123.698 90)
+			(at 162.306 144.018 90)
 			(effects
 				(font
@@
 		)
 		(property "Footprint" "Resistor_SMD:R_0603_1608Metric_Pad0.98x0.95mm_HandSolder"
-			(at 158.242 121.92 90)
+			(at 158.242 142.24 90)
 			(effects
 				(font
@@
 		)
 		(property "Datasheet" "~"
-			(at 160.02 121.92 0)
-			(effects
-				(font
-					(size 1.27 1.27)
-				)
-			)
-		)
-		(property "Description" ""
-			(at 160.02 121.92 0)
-			(effects
-				(font
+			(at 160.02 142.24 0)
+			(effects
+				(font
+					(size 1.27 1.27)
+				)
+			)
+		)
+		(property "Description" ""
+			(at 160.02 142.24 0)
+			(effects
+				(font
