File: Power_Amp.kicad_sch (KiCad schematic)
At the start: 34 parts, among them J10 2118718-2, P13 CONUFL001-SMD-T, U27 TQP7M9106, U28 ADL5501AKSZ, U29 ADL5501AKSZ

Commit message: More work on components
Signed-off-by: Corey Minyard <corey@minyard.net>
Parts:
- removed H20, H21: Wire_Hole, PacSatDev_misc:Wire_Hole, symbol PACSAT_DEV_misc:CUBESAT_MOUNT_HOLE_1
- added J17: Conn_01x02_Pin, Connector_Wire:SolderWire-0.5sqmm_1x02_P4.6mm_D0.9mm_OD2.1mm, symbol Connector:Conn_01x02_Pin
- C112: value 100p -> 1n
- C117: value 114p 2% 30V -> 110p 1% 30V
- C123: value 100p 30V -> 1n
- L35: value 17n 2% Q>=40 -> 18n 2% Q=58
Connections:
- net GND: now also J17.1 (Pin_1), J17.2 (Pin_2)
Changed lines of the file:
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@@
 	)
 	(junction
+		(at 267.97 107.95)
+		(diameter 0)
+		(color 0 0 0 0)
+	)
+	(junction
 		(at 124.46 40.64)
 		(diameter 0)
@@
 	)
 	(junction
-		(at 267.97 114.3)
-		(diameter 0)
-		(color 0 0 0 0)
-	)
-	(junction
 		(at 147.32 142.24)
 		(diameter 0)
@@
 	(wire
 		(pts
-			(xy 252.73 114.3) (xy 267.97 114.3)
-		)
-		(stroke
-			(width 0)
-			(type default)
-		)
-	)
-	(wire
-		(pts
 			(xy 83.82 160.02) (xy 83.82 162.56)
 		)
@@
 	(wire
 		(pts
+			(xy 252.73 107.95) (xy 267.97 107.95)
+		)
+		(stroke
+			(width 0)
+			(type default)
+		)
+	)
+	(wire
+		(pts
 			(xy 147.32 147.32) (xy 147.32 149.86)
 		)
@@
 	(wire
 		(pts
-			(xy 267.97 114.3) (xy 267.97 116.84)
+			(xy 267.97 107.95) (xy 267.97 116.84)
 		)
 		(stroke
@@
 	(wire
 		(pts
-			(xy 267.97 105.41) (xy 267.97 114.3)
+			(xy 267.97 105.41) (xy 267.97 107.95)
 		)
 		(stroke
@@
 	)
 	(symbol
-		(lib_id "PACSAT_DEV_misc:CUBESAT_MOUNT_HOLE_1")
-		(at 250.19 105.41 0)
-		(unit 1)
-		(exclude_from_sim no)
-		(in_bom no)
-		(on_board yes)
-		(dnp no)
-		(property "Reference" "H20"
-			(at 250.9774 99.3902 0)
-			(effects
-				(font
-					(size 1.524 1.524)
-				)
-			)
-		)
-		(property "Value" "Wire_Hole"
-			(at 250.9774 102.0826 0)
-			(effects
-				(font
-					(size 1.524 1.524)
-				)
-			)
-		)
-		(property "Footprint" "PacSatDev_misc:Wire_Hole"
-			(at 250.19 105.41 0)
-			(effects
-				(font
-					(size 1.524 1.524)
-				)
-				(hide yes)
-			)
-		)
-		(property "Datasheet" ""
-			(at 250.19 105.41 0)
-			(effects
-				(font
-					(size 1.524 1.524)
-				)
-				(hide yes)
-			)
-		)
-		(property "Description" ""
-			(at 250.19 105.41 0)
-			(effects
-				(font
-					(size 1.27 1.27)
-				)
-			)
-		)
-		(pin "1"
-		)
-		(instances
-			(project "PacSat_AFSK"
-				(path "/cc9f42d2-6985-41ac-acab-5ab7b01c5b38/b85b88c3-87c5-49e2-804e-0759552ace3d"
-					(reference "H20")
-					(unit 1)
-				)
-			)
-		)
-	)
-	(symbol
 		(lib_id "power:GND")
 		(at 163.83 228.6 0)
@@
 	)
 	(symbol
-		(lib_id "PACSAT_DEV_misc:CUBESAT_MOUNT_HOLE_1")
-		(at 250.19 114.3 0)
-		(unit 1)
-		(exclude_from_sim no)
-		(in_bom no)
-		(on_board yes)
-		(dnp no)
-		(property "Reference" "H21"
-			(at 250.9774 108.2802 0)
-			(effects
-				(font
-					(size 1.524 1.524)
-				)
-			)
-		)
-		(property "Value" "Wire_Hole"
-			(at 250.9774 110.9726 0)
-			(effects
-				(font
-					(size 1.524 1.524)
-				)
-			)
-		)
-		(property "Footprint" "PacSatDev_misc:Wire_Hole"
-			(at 250.19 114.3 0)
-			(effects
-				(font
-					(size 1.524 1.524)
-				)
-				(hide yes)
-			)
-		)
-		(property "Datasheet" ""
-			(at 250.19 114.3 0)
-			(effects
-				(font
-					(size 1.524 1.524)
-				)
-				(hide yes)
-			)
-		)
-		(property "Description" ""
-			(at 250.19 114.3 0)
-			(effects
-				(font
-					(size 1.27 1.27)
-				)
-			)
-		)
-		(pin "1"
-		)
-		(instances
-			(project "PacSat_AFSK"
-				(path "/cc9f42d2-6985-41ac-acab-5ab7b01c5b38/b85b88c3-87c5-49e2-804e-0759552ace3d"
-					(reference "H21")
-					(unit 1)
-				)
-			)
-		)
-	)
-	(symbol
 		(lib_id "Device:L")
 		(at 255.27 148.59 90)
@@
 			)
 		)
-		(property "Value" "100p 30V"
+		(property "Value" "1n"
 			(at 199.39 156.718 90)
 			(effects
@@
 			)
 		)
-		(property "Value" "114p 2% 30V"
+		(property "Value" "110p 1% 30V"
 			(at 217.17 163.322 90)
 			(effects
@@
 	)
 	(symbol
+		(lib_id "Connector:Conn_01x02_Pin")
+		(at 247.65 105.41 0)
+		(unit 1)
+		(exclude_from_sim no)
+		(in_bom no)
+		(on_board yes)
+		(dnp no)
+		(fields_autoplaced yes)
+		(property "Reference" "J17"
+			(at 248.285 100.33 0)
+			(effects
+				(font
+					(size 1.27 1.27)
+				)
+			)
+		)
+		(property "Value" "Conn_01x02_Pin"
+			(at 248.285 102.87 0)
+			(effects
+				(font
+					(size 1.27 1.27)
+				)
+			)
+		)
+		(property "Footprint" "Connector_Wire:SolderWire-0.5sqmm_1x02_P4.6mm_D0.9mm_OD2.1mm"
+			(at 247.65 105.41 0)
+			(effects
+				(font
+					(size 1.27 1.27)
+				)
+				(hide yes)
+			)
+		)
+		(property "Datasheet" "~"
+			(at 247.65 105.41 0)
+			(effects
+				(font
+					(size 1.27 1.27)
+				)
+				(hide yes)
+			)
+		)
+		(property "Description" "Generic connector, single row, 01x02, script generated"
+			(at 247.65 105.41 0)
+			(effects
+				(font
+					(size 1.27 1.27)
+				)
+				(hide yes)
+			)
+		)
+		(pin "1"
+		)
+		(pin "2"
+		)
+		(instances
+			(project "PacSat_AFSK"
+				(path "/cc9f42d2-6985-41ac-acab-5ab7b01c5b38/b85b88c3-87c5-49e2-804e-0759552ace3d"
+					(reference "J17")
+					(unit 1)
+				)
+			)
+		)
+	)
+	(symbol
 		(lib_id "Device:C")
 		(at 214.63 125.73 0)
@@
 			)
 		)
-		(property "Value" "100p"
+		(property "Value" "1n"
 			(at 45.72 138.43 90)
 			(effects
@@
 			)
 		)
-		(property "Value" "17n 2% Q>=40"
+		(property "Value" "18n 2% Q=58"
 			(at 62.484 140.208 90)
 			(effects

Commit message: More work on simulation and component choice
Signed-off-by: Corey Minyard <corey@minyard.net>
Parts:
- L35: value 18n 2% Q=58 -> 18n 2% Q=80
Changed lines of the file:
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@@
 			)
 		)
-		(property "Value" "18n 2% Q=58"
+		(property "Value" "18n 2% Q=80"
 			(at 62.484 140.208 90)
 			(effects

Commit message: Lots of updates to ease manufacturing
Component changes, changes in the formatting of the values, etc.

Signed-off-by: Corey Minyard <corey@minyard.net>
Parts:
- C101, C112, C116, C119, C123: value 1n -> 1nF
- C113, C115: value 100p -> 100pF
- C114: value 39p 1% -> 39pF 1%
- C117: value 110p 1% 30V -> 110pF 1% 30V
- C118: value 10u -> 10uF
- C124: value 7.3p 2% 30V -> 7.3pF 2% 30V
- C125: value 0.75p 2% 30V -> 0.75pF 2% 30V
- C126: value 12p 2% 30v -> 12pF 2% 30v
- C127: value 2.2p 2% 30v -> 2.2pF 2% 30v
- C128: value 6.2p 2% 30v -> 6.2pF 2% 30v
- L30: value 22n 2% Q=67 -> 22nH 2% Q=67
- L33: value 18n 2% Q=58 -> 18nH 2% Q=58
- L35: value 18n 2% Q=80 -> 18nH 2% Q=80
- L36: value 68n -> 68nH
- L37: value 36n Q=79 I>1A -> 36nH Q=79 I>1A
- L38: value 6.9n 2% Q=69 -> 6.9nH 2% Q=69
- U28, U29: value ADL5501AKSZ -> ADL5501AKSZ-R7
Other:
- note added: "Thermsistor varies from 500 ohms (125C) to 350K (-50C). With a 10K bias this gives a .16 to 3.2V range."
- note removed: "Thermsistor varies from 500 ohms (125C) to 350k (-50C). With a 10K bias this gives a .16 to 3.2V range."
- moved on the sheet: C127, C128, L33
Changed lines of the file:
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@@
 		)
 	)
-	(text "Thermsistor varies from 500\nohms (125C) to 350k (-50C).\nWith a 10K bias this gives a\n.16 to 3.2V range."
+	(text "Thermsistor varies from 500\nohms (125C) to 350K (-50C).\nWith a 10K bias this gives a\n.16 to 3.2V range."
 		(exclude_from_sim no)
 		(at 142.494 205.232 0)
@@
 	)
 	(junction
-		(at 266.7 160.02)
-		(diameter 0)
-		(color 0 0 0 0)
-	)
-	(junction
 		(at 124.46 38.1)
 		(diameter 0)
@@
 	)
 	(junction
-		(at 285.75 160.02)
+		(at 283.21 160.02)
 		(diameter 0)
 		(color 0 0 0 0)
@@
 	)
 	(junction
+		(at 264.16 148.59)
+		(diameter 0)
+		(color 0 0 0 0)
+	)
+	(junction
 		(at 124.46 68.58)
 		(diameter 0)
@@
 	(wire
 		(pts
-			(xy 273.05 148.59) (xy 266.7 148.59)
+			(xy 270.51 148.59) (xy 264.16 148.59)
 		)
 		(stroke
@@
 	(wire
 		(pts
-			(xy 285.75 160.02) (xy 280.67 160.02)
+			(xy 283.21 160.02) (xy 278.13 160.02)
 		)
 		(stroke
@@
 	(wire
 		(pts
-			(xy 285.75 173.99) (xy 285.75 179.07)
+			(xy 283.21 173.99) (xy 283.21 179.07)
 		)
 		(stroke
@@
 	(wire
 		(pts
-			(xy 285.75 148.59) (xy 285.75 160.02)
+			(xy 283.21 148.59) (xy 283.21 160.02)
 		)
 		(stroke
@@
 	(wire
 		(pts
-			(xy 285.75 160.02) (xy 285.75 166.37)
+			(xy 283.21 160.02) (xy 283.21 166.37)
 		)
 		(stroke
@@
 	(wire
 		(pts
-			(xy 264.16 160.02) (xy 266.7 160.02)
-		)
-		(stroke
-			(width 0)
-			(type default)
-		)
-	)
-	(wire
-		(pts
 			(xy 124.46 66.04) (xy 124.46 68.58)
 		)
@@
 	(wire
 		(pts
-			(xy 280.67 148.59) (xy 285.75 148.59)
+			(xy 278.13 148.59) (xy 283.21 148.59)
 		)
 		(stroke
@@
 	(wire
 		(pts
-			(xy 266.7 148.59) (xy 266.7 160.02)
+			(xy 264.16 160.02) (xy 270.51 160.02)
 		)
 		(stroke
@@
 	(wire
 		(pts
-			(xy 266.7 160.02) (xy 273.05 160.02)
-		)
-		(stroke
-			(width 0)
-			(type default)
-		)
-	)
-	(wire
-		(pts
 			(xy 398.78 100.33) (xy 405.13 100.33)
 		)
@@
 	(wire
 		(pts
-			(xy 285.75 160.02) (xy 302.26 160.02)
+			(xy 283.21 160.02) (xy 302.26 160.02)
 		)
 		(stroke
@@
 	(symbol
 		(lib_id "Device:L")
-		(at 276.86 148.59 90)
+		(at 274.32 148.59 90)
 		(mirror x)
 		(unit 1)
@@
 		(dnp no)
 		(property "Reference" "L33"
-			(at 276.86 146.812 90)
+			(at 274.32 146.812 90)
 			(effects
 				(font
@@
 			)
 		)
-		(property "Value" "18n 2% Q=58"
-			(at 276.86 150.622 90)
+		(property "Value" "18nH 2% Q=58"
+			(at 274.32 150.622 90)
 			(effects
 				(font
@@
 		)
 		(property "Footprint" "Inductor_SMD:L_0402_1005Metric_Pad0.77x0.64mm_HandSolder"
-			(at 276.86 148.59 0)
+			(at 274.32 148.59 0)
 			(effects
 				(font
@@
 		)
 		(property "Datasheet" "~"
-			(at 276.86 148.59 0)
+			(at 274.32 148.59 0)
 			(effects
 				(font
@@
 		)
 		(property "Description" ""
-			(at 276.86 148.59 0)
+			(at 274.32 148.59 0)
 			(effects
 				(font
@@
 			)
 		)
-		(property "Value" "100p"
+		(property "Value" "100pF"
 			(at 201.93 133.35 0)
 			(effects
@@
 	(symbol
 		(lib_id "Device:C")
-		(at 285.75 170.18 180)
+		(at 283.21 170.18 180)
 		(unit 1)
 		(exclude_from_sim no)
@@
 		(dnp no)
 		(property "Reference" "C128"
-			(at 282.194 169.672 90)
+			(at 279.654 169.672 90)
 			(effects
 				(font
@@
 			)
 		)
-		(property "Value" "6.2p 2% 30v"
-			(at 289.052 169.926 90)
+		(property "Value" "6.2pF 2% 30v"
+			(at 286.512 169.926 90)
 			(effects
 				(font
@@
 		)
 		(property "Footprint" "Capacitor_SMD:C_0402_1005Metric_Pad0.74x0.62mm_HandSolder"
-			(at 284.7848 166.37 0)
+			(at 282.2448 166.37 0)
 			(effects
 				(font
@@
 		)
 		(property "Datasheet" "~"
-			(at 285.75 170.18 0)
+			(at 283.21 170.18 0)
 			(effects
 				(font
@@
 		)
 		(property "Description" ""
-			(at 285.75 170.18 0)
+			(at 283.21 170.18 0)
 			(effects
 				(font
@@
 			)
 		)
-		(property "Value" "68n"
+		(property "Value" "68nH"
 			(at 157.226 121.158 90)
 			(effects
@@
 			)
 		)
-		(property "Value" "39p 1%"
+		(property "Value" "39pF 1%"
 			(at 64.77 154.94 0)
 			(effects
@@
 			)
 		)
-		(property "Value" "ADL5501AKSZ"
+		(property "Value" "ADL5501AKSZ-R7"
 			(at 314.96 90.17 0)
 			(effects
@@
 			)
 		)
-		(property "Value" "12p 2% 30v"
+		(property "Value" "12pF 2% 30v"
 			(at 267.462 169.926 90)
 			(effects
@@
 			)
 		)
-		(property "Value" "22n 2% Q=67"
+		(property "Value" "22nH 2% Q=67"
 			(at 255.27 150.622 90)
 			(effects
@@
 			)
 		)
-		(property "Value" "100p"
+		(property "Value" "100pF"
 			(at 74.93 120.65 0)
 			(effects
@@
 			)
 		)
-		(property "Value" "1n"
+		(property "Value" "1nF"
 			(at 199.39 156.718 90)
 			(effects
@@
 			)
 		)
-		(property "Value" "110p 1% 30V"
+		(property "Value" "110pF 1% 30V"
 			(at 217.17 163.322 90)
 			(effects
@@
 			)
 		)
-		(property "Value" "10u"
+		(property "Value" "10uF"
 			(at 218.44 110.49 0)
 			(effects
@@
 			)
 		)
-		(property "Value" "1n"
+		(property "Value" "1nF"
 			(at 208.28 120.65 0)
 			(effects
@@
 			)
 		)
-		(property "Value" "1n"
+		(property "Value" "1nF"
 			(at 344.678 95.25 90)
 			(effects
@@
 			)
 		)
-		(property "Value" "6.9n 2% Q=69"
+		(property "Value" "6.9nH 2% Q=69"
 			(at 230.632 170.18 90)
 			(effects
@@
 			)
 		)
-		(property "Value" "0.75p 2% 30V"
+		(property "Value" "0.75pF 2% 30V"
 			(at 255.524 156.464 90)
 			(effects
@@
 			)
 		)
-		(property "Value" "36n Q=79 I>1A"
+		(property "Value" "36nH Q=79 I>1A"
 			(at 191.77 140.716 90)
 			(effects
@@
 			)
 		)
-		(property "Value" "1n"
+		(property "Value" "1nF"
 			(at 281.178 95.25 90)
 			(effects
@@
 			)
 		)
-		(property "Value" "ADL5501AKSZ"
+		(property "Value" "ADL5501AKSZ-R7"
 			(at 378.46 90.17 0)
 			(effects
@@
 	(symbol
 		(lib_id "Device:C")
-		(at 276.86 160.02 90)
+		(at 274.32 160.02 90)
 		(unit 1)
 		(exclude_from_sim no)
@@
 		(dnp no)
 		(property "Reference" "C127"
-			(at 277.114 153.924 90)
+			(at 274.574 153.924 90)
 			(effects
 				(font
@@
 			)
 		)
-		(property "Value" "2.2p 2% 30v"
-			(at 277.114 156.464 90)
+		(property "Value" "2.2pF 2% 30v"
+			(at 274.574 156.464 90)
 			(effects
 				(font
@@
 		)
 		(property "Footprint" "Capacitor_SMD:C_0402_1005Metric_Pad0.74x0.62mm_HandSolder"
-			(at 280.67 159.0548 0)
+			(at 278.13 159.0548 0)
 			(effects
 				(font
@@
 		)
 		(property "Datasheet" "~"
-			(at 276.86 160.02 0)
+			(at 274.32 160.02 0)
 			(effects
 				(font
@@
 		)
 		(property "Description" ""
-			(at 276.86 160.02 0)
+			(at 274.32 160.02 0)
 			(effects
 				(font
@@
 	(symbol
 		(lib_id "power:GND")
-		(at 285.75 179.07 0)
+		(at 283.21 179.07 0)
 		(unit 1)
 		(exclude_from_sim no)
@@
 		(dnp no)
 		(property "Reference" "#PWR0291"
-			(at 285.75 185.42 0)
+			(at 283.21 185.42 0)
 			(effects
 				(font
@@
 		)
 		(property "Value" "GND"
-			(at 285.877 183.4642 0)
+			(at 283.337 183.4642 0)
 			(effects
 				(font
@@
 		)
 		(property "Footprint" ""
-			(at 285.75 179.07 0)
+			(at 283.21 179.07 0)
 			(effects
 				(font
@@
 		)
 		(property "Datasheet" ""
-			(at 285.75 179.07 0)
+			(at 283.21 179.07 0)
 			(effects
 				(font
@@
 		)
 		(property "Description" ""
-			(at 285.75 179.07 0)
+			(at 283.21 179.07 0)
 			(effects
 				(font
@@
 			)
 		)
-		(property "Value" "7.3p 2% 30V"
+		(property "Value" "7.3pF 2% 30V"
 			(at 248.412 169.926 90)
 			(effects
@@
 			)
 		)
-		(property "Value" "1n"
+		(property "Value" "1nF"
 			(at 45.72 138.43 90)
 			(effects
@@
 			)
 		)
-		(property "Value" "18n 2% Q=80"
-			(at 62.484 140.208 90)
+		(property "Value" "18nH 2% Q=80"
+			(at 65.278 139.954 90)
 			(effects
 				(font

Commit message: Update all resistors to have an ohm symbol
Make it more clean in the BOM what they are.

Signed-off-by: Corey Minyard <corey@minyard.net>
Parts:
- R78: value 280 -> 280Ω
- R79: value 240 -> 240Ω
- R80, R82: value 49.9 -> 50Ω
- R81: value 10K 1% -> 10KΩ 1%
Other:
- note added: "Thermsistor varies from 500 ohms (125C) to 350KΩ (-50C). With a 10KΩ bias this gives a .16 to 3.2V range."
- note removed: "Thermsistor varies from 500 ohms (125C) to 350K (-50C). With a 10K bias this gives a .16 to 3.2V range."
Changed lines of the file:
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@@
 		)
 	)
-	(text "Thermsistor varies from 500\nohms (125C) to 350K (-50C).\nWith a 10K bias this gives a\n.16 to 3.2V range."
+	(text "Thermsistor varies from 500\nohms (125C) to 350KΩ (-50C).\nWith a 10KΩ bias this gives a\n.16 to 3.2V range."
 		(exclude_from_sim no)
 		(at 142.494 205.232 0)
@@
 			)
 		)
-		(property "Value" "49.9"
+		(property "Value" "50Ω"
 			(at 371.856 147.828 90)
 			(effects
@@
 			)
 		)
-		(property "Value" "280"
+		(property "Value" "280Ω"
 			(at 84.836 109.728 90)
 			(effects
@@
 			)
 		)
-		(property "Value" "10K 1%"
+		(property "Value" "10KΩ 1%"
 			(at 153.924 211.582 0)
 			(effects
@@
 			)
 		)
-		(property "Value" "240"
+		(property "Value" "240Ω"
 			(at 162.306 144.018 90)
 			(effects
@@
 			)
 		)
-		(property "Value" "49.9"
+		(property "Value" "50Ω"
 			(at 318.516 147.828 90)
 			(effects

Commit message: Massive rework of filtering and inductors
Now that I know how inductors really work.

Signed-off-by: Corey Minyard <corey@minyard.net>
Parts:
- L30: value 22nH 2% Q=67 -> 22nH 2%
- L33: value 18nH 2% Q=58 -> 18nH 2%
- L35: value 18nH 2% Q=80 -> 18nH 2%
- L37: value 36nH Q=79 I>1A -> 36nH I>1A
- L38: value 6.9nH 2% Q=69 -> 6.9nH 2%
Other:
- note added: "-2 dB"
- note removed: "-1.3 dB"
- moved on the sheet: C117
Changed lines of the file:
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@@
 		)
 	)
-	(text "-1.3 dB"
+	(text "-2 dB"
 		(exclude_from_sim no)
 		(at 260.858 141.986 0)
@@
 	(wire
 		(pts
-			(xy 220.98 160.02) (xy 228.6 160.02)
+			(xy 224.79 160.02) (xy 228.6 160.02)
 		)
 		(stroke
@@
 	(wire
 		(pts
-			(xy 203.2 160.02) (xy 213.36 160.02)
+			(xy 203.2 160.02) (xy 217.17 160.02)
 		)
 		(stroke
@@
 			)
 		)
-		(property "Value" "18nH 2% Q=58"
+		(property "Value" "18nH 2%"
 			(at 274.32 150.622 90)
 			(effects
@@
 			)
 		)
-		(property "Value" "22nH 2% Q=67"
+		(property "Value" "22nH 2%"
 			(at 255.27 150.622 90)
 			(effects
@@
 	(symbol
 		(lib_id "Device:C")
-		(at 217.17 160.02 270)
+		(at 220.98 160.02 270)
 		(mirror x)
 		(unit 1)
@@
 		(dnp no)
 		(property "Reference" "C117"
-			(at 217.17 156.21 90)
+			(at 220.98 156.21 90)
 			(effects
 				(font
@@
 		)
 		(property "Value" "110pF 1% 30V"
-			(at 217.17 163.322 90)
+			(at 220.98 163.322 90)
 			(effects
 				(font
@@
 		)
 		(property "Footprint" "Capacitor_SMD:C_0402_1005Metric_Pad0.74x0.62mm_HandSolder"
-			(at 213.36 159.0548 0)
+			(at 217.17 159.0548 0)
 			(effects
 				(font
@@
 		)
 		(property "Datasheet" "~"
-			(at 217.17 160.02 0)
+			(at 220.98 160.02 0)
 			(effects
 				(font
@@
 		)
 		(property "Description" ""
-			(at 217.17 160.02 0)
+			(at 220.98 160.02 0)
 			(effects
 				(font
@@
 			)
 		)
-		(property "Value" "6.9nH 2% Q=69"
+		(property "Value" "6.9nH 2%"
 			(at 230.632 170.18 90)
 			(effects
@@
 			)
 		)
-		(property "Value" "36nH Q=79 I>1A"
+		(property "Value" "36nH I>1A"
 			(at 191.77 140.716 90)
 			(effects
@@
 			)
 		)
-		(property "Value" "18nH 2% Q=80"
+		(property "Value" "18nH 2%"
 			(at 65.278 139.954 90)
 			(effects

Commit message: Take into account capacitance of inductors
Signed-off-by: Corey Minyard <corey@minyard.net>
Parts:
- L33: value 18nH 2% -> 18nH 2% 0402
Changed lines of the file:
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@@
 	(text "-2 dB"
 		(exclude_from_sim no)
-		(at 260.858 141.986 0)
+		(at 243.078 142.494 0)
 		(effects
 			(font
@@
 			)
 		)
-		(property "Value" "18nH 2%"
+		(property "Value" "18nH 2% 0402"
 			(at 274.32 150.622 90)
 			(effects

Commit message: Rework PA input impedance match
The two inductor L match works better than the LC match.

Signed-off-by: Corey Minyard <corey@minyard.net>
Parts:
- removed C114: 39pF 1%, Capacitor_SMD:C_0402_1005Metric_Pad0.74x0.62mm_HandSolder, symbol Device:C
- added L27: 3.3nH 2%, Inductor_SMD:L_0603_1608Metric_Pad1.05x0.95mm_HandSolder, symbol Device:L
- L35: value 18nH 2% -> 11nH 2%
Connections:
- net GND: now also L27.1
- net at C112.2, L35.1, P13.1 (In): now also L27.2
Changed lines of the file:
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@@
 	(symbol
 		(lib_id "Device:L")
+		(at 58.42 152.4 180)
+		(unit 1)
+		(exclude_from_sim no)
+		(in_bom yes)
+		(on_board yes)
+		(dnp no)
+		(property "Reference" "L27"
+			(at 60.198 152.4 90)
+			(effects
+				(font
+					(size 1.27 1.27)
+				)
+			)
+		)
+		(property "Value" "3.3nH 2%"
+			(at 56.134 153.162 90)
+			(effects
+				(font
+					(size 1.27 1.27)
+				)
+			)
+		)
+		(property "Footprint" "Inductor_SMD:L_0603_1608Metric_Pad1.05x0.95mm_HandSolder"
+			(at 58.42 152.4 0)
+			(effects
+				(font
+					(size 1.27 1.27)
+				)
+				(hide yes)
+			)
+		)
+		(property "Datasheet" "~"
+			(at 58.42 152.4 0)
+			(effects
+				(font
+					(size 1.27 1.27)
+				)
+				(hide yes)
+			)
+		)
+		(property "Description" ""
+			(at 58.42 152.4 0)
+			(effects
+				(font
+					(size 1.27 1.27)
+				)
+			)
+		)
+		(pin "1"
+		)
+		(pin "2"
+		)
+		(instances
+			(project "PacSat_AFSK"
+				(path "/cc9f42d2-6985-41ac-acab-5ab7b01c5b38/b85b88c3-87c5-49e2-804e-0759552ace3d"
+					(reference "L27")
+					(unit 1)
+				)
+			)
+		)
+	)
+	(symbol
+		(lib_id "Device:L")
 		(at 160.02 121.92 180)
 		(unit 1)
@@
 	)
 	(symbol
-		(lib_id "Device:C")
-		(at 58.42 152.4 0)
-		(unit 1)
-		(exclude_from_sim no)
-		(in_bom yes)
-		(on_board yes)
-		(dnp no)
-		(property "Reference" "C114"
-			(at 63.5 152.4 0)
-			(effects
-				(font
-					(size 1.27 1.27)
-				)
-			)
-		)
-		(property "Value" "39pF 1%"
-			(at 64.77 154.94 0)
-			(effects
-				(font
-					(size 1.27 1.27)
-				)
-			)
-		)
-		(property "Footprint" "Capacitor_SMD:C_0402_1005Metric_Pad0.74x0.62mm_HandSolder"
-			(at 59.3852 156.21 0)
-			(effects
-				(font
-					(size 1.27 1.27)
-				)
-				(hide yes)
-			)
-		)
-		(property "Datasheet" "~"
-			(at 58.42 152.4 0)
-			(effects
-				(font
-					(size 1.27 1.27)
-				)
-				(hide yes)
-			)
-		)
-		(property "Description" ""
-			(at 58.42 152.4 0)
-			(effects
-				(font
-					(size 1.27 1.27)
-				)
-			)
-		)
-		(pin "1"
-		)
-		(pin "2"
-		)
-		(instances
-			(project "PacSat_AFSK"
-				(path "/cc9f42d2-6985-41ac-acab-5ab7b01c5b38/b85b88c3-87c5-49e2-804e-0759552ace3d"
-					(reference "C114")
-					(unit 1)
-				)
-			)
-		)
-	)
-	(symbol
 		(lib_id "power:GND")
 		(at 54.61 124.46 0)
@@
 			)
 		)
-		(property "Value" "18nH 2%"
+		(property "Value" "11nH 2%"
 			(at 65.278 139.954 90)
 			(effects

Commit message: Minor fixes for BOM values
Signed-off-by: Corey Minyard <corey@minyard.net>
Parts:
- TH4: value NCU15XH103F60RC 10K@25C -> NCU15XH103F60RC 10KΩ@25C
Changed lines of the file:
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@@
 			)
 		)
-		(property "Value" "NCU15XH103F60RC 10K@25C"
+		(property "Value" "NCU15XH103F60RC 10KΩ@25C"
 			(at 171.196 231.394 90)
 			(effects
