File: RX_2_ax5043.kicad_sch (KiCad schematic)
At the start: 19 parts, among them J3 2118714-2, P2 CONUFL001-SMD-T, Q4 DMP2037U, U15 AX5043

Commit message: Change appropriate passives to 0402 on the receive AX5043s
Signed-off-by: Corey Minyard <corey@minyard.net>
Parts:
- C49: footprint Resistor_SMD:R_0603_1608Metric_Pad0.98x0.95mm_HandSolder -> Capacitor_SMD:C_0402_1005Metric_Pad0.74x0.62mm_HandSolder
- C50, C51, C53, C54, C55, C56: footprint Capacitor_SMD:C_0603_1608Metric_Pad1.08x0.95mm_HandSolder -> Capacitor_SMD:C_0402_1005Metric_Pad0.74x0.62mm_HandSolder
- R52, R55: footprint Resistor_SMD:R_0603_1608Metric_Pad0.98x0.95mm_HandSolder -> Resistor_SMD:R_0402_1005Metric_Pad0.72x0.64mm_HandSolder
Changed lines of the file:
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@@
 			)
 		)
-		(property "Footprint" "Capacitor_SMD:C_0603_1608Metric_Pad1.08x0.95mm_HandSolder"
+		(property "Footprint" "Capacitor_SMD:C_0402_1005Metric_Pad0.74x0.62mm_HandSolder"
 			(at 211.7852 93.98 0)
 			(effects
@@
 			)
 		)
-		(property "Footprint" "Capacitor_SMD:C_0603_1608Metric_Pad1.08x0.95mm_HandSolder"
+		(property "Footprint" "Capacitor_SMD:C_0402_1005Metric_Pad0.74x0.62mm_HandSolder"
 			(at 148.8948 135.89 0)
 			(effects
@@
 			)
 		)
-		(property "Footprint" "Capacitor_SMD:C_0603_1608Metric_Pad1.08x0.95mm_HandSolder"
+		(property "Footprint" "Capacitor_SMD:C_0402_1005Metric_Pad0.74x0.62mm_HandSolder"
 			(at 192.7352 90.17 0)
 			(effects
@@
 			)
 		)
-		(property "Footprint" "Capacitor_SMD:C_0603_1608Metric_Pad1.08x0.95mm_HandSolder"
+		(property "Footprint" "Capacitor_SMD:C_0402_1005Metric_Pad0.74x0.62mm_HandSolder"
 			(at 188.9252 151.13 0)
 			(effects
@@
 			)
 		)
-		(property "Footprint" "Capacitor_SMD:C_0603_1608Metric_Pad1.08x0.95mm_HandSolder"
+		(property "Footprint" "Capacitor_SMD:C_0402_1005Metric_Pad0.74x0.62mm_HandSolder"
 			(at 243.5352 102.87 0)
 			(effects
@@
 			)
 		)
-		(property "Footprint" "Resistor_SMD:R_0603_1608Metric_Pad0.98x0.95mm_HandSolder"
+		(property "Footprint" "Resistor_SMD:R_0402_1005Metric_Pad0.72x0.64mm_HandSolder"
 			(at 255.27 138.938 90)
 			(effects
@@
 			)
 		)
-		(property "Footprint" "Capacitor_SMD:C_0603_1608Metric_Pad1.08x0.95mm_HandSolder"
+		(property "Footprint" "Capacitor_SMD:C_0402_1005Metric_Pad0.74x0.62mm_HandSolder"
 			(at 137.16 134.3152 0)
 			(effects
@@
 			)
 		)
-		(property "Footprint" "Resistor_SMD:R_0603_1608Metric_Pad0.98x0.95mm_HandSolder"
+		(property "Footprint" "Capacitor_SMD:C_0402_1005Metric_Pad0.74x0.62mm_HandSolder"
 			(at 131.7752 118.11 0)
 			(effects
@@
 			)
 		)
-		(property "Footprint" "Resistor_SMD:R_0603_1608Metric_Pad0.98x0.95mm_HandSolder"
+		(property "Footprint" "Resistor_SMD:R_0402_1005Metric_Pad0.72x0.64mm_HandSolder"
 			(at 174.752 143.51 90)
 			(effects

Commit message: Work on cleaning up all values for things
Signed-off-by: Corey Minyard <corey@minyard.net>
Parts:
- C50, C51: value 15p -> 15p 1%
- L3, L4: value 78n -> 78n 2% Q=28
- L5: value 1n -> 1n Q=77; footprint Inductor_SMD:L_0603_1608Metric_Pad1.05x0.95mm_HandSolder -> Inductor_SMD:L_0402_1005Metric_Pad0.77x0.64mm_HandSolder
Changed lines of the file:
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@@
 			)
 		)
-		(property "Value" "1n"
+		(property "Value" "1n Q=77"
 			(at 171.704 139.446 90)
 			(effects
@@
 			)
 		)
-		(property "Footprint" "Inductor_SMD:L_0603_1608Metric_Pad1.05x0.95mm_HandSolder"
+		(property "Footprint" "Inductor_SMD:L_0402_1005Metric_Pad0.77x0.64mm_HandSolder"
 			(at 170.18 139.7 0)
 			(effects
@@
 			)
 		)
-		(property "Value" "15p"
+		(property "Value" "15p 1%"
 			(at 152.4 143.51 90)
 			(effects
@@
 			)
 		)
-		(property "Value" "78n"
+		(property "Value" "78n 2% Q=28"
 			(at 161.798 139.7 90)
 			(effects
@@
 			)
 		)
-		(property "Value" "15p"
+		(property "Value" "15p 1%"
 			(at 144.78 130.81 90)
 			(effects
@@
 			)
 		)
-		(property "Value" "78n"
+		(property "Value" "78n 2% Q=28"
 			(at 139.7 125.222 90)
 			(effects

Commit message: More work on components
Signed-off-by: Corey Minyard <corey@minyard.net>
Parts:
- FB5: value 1K @ 100MHz -> 1K@100MHz
Changed lines of the file:
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@@
 			)
 		)
-		(property "Value" "1K @ 100MHz"
+		(property "Value" "1K@100MHz"
 			(at 266.6619 66.04 90)
 			(effects

Commit message: Lots of updates to ease manufacturing
Component changes, changes in the formatting of the values, etc.

Signed-off-by: Corey Minyard <corey@minyard.net>
Parts:
- C49: value 100p -> 100pF
- C50, C51: value 15p 1% -> 15pF 1%
- C52, C53, C56: value 10n -> 10nF
- C54: value 6.8p -> 6.8pF
- C55: value 10p -> 10pF
- L3, L4: value 78n 2% Q=28 -> 78nH 2% Q=28
- L5: value 1n Q=77 -> 1nH Q=77
- Q4: value DMP2037U -> DMP2037U-7
Changed lines of the file:
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@@
 			)
 		)
-		(property "Value" "10p"
+		(property "Value" "10pF"
 			(at 214.63 87.63 90)
 			(effects
@@
 			)
 		)
-		(property "Value" "1n Q=77"
+		(property "Value" "1nH Q=77"
 			(at 171.704 139.446 90)
 			(effects
@@
 			)
 		)
-		(property "Value" "15p 1%"
+		(property "Value" "15pF 1%"
 			(at 152.4 143.51 90)
 			(effects
@@
 			)
 		)
-		(property "Value" "78n 2% Q=28"
+		(property "Value" "78nH 2% Q=28"
 			(at 161.798 139.7 90)
 			(effects
@@
 			)
 		)
-		(property "Value" "6.8p"
+		(property "Value" "6.8pF"
 			(at 195.58 83.82 90)
 			(effects
@@
 			)
 		)
-		(property "Value" "10n"
+		(property "Value" "10nF"
 			(at 187.96 110.49 90)
 			(effects
@@
 			)
 		)
-		(property "Value" "10n"
+		(property "Value" "10nF"
 			(at 185.42 143.51 90)
 			(effects
@@
 			)
 		)
-		(property "Value" "10n"
+		(property "Value" "10nF"
 			(at 246.38 96.52 90)
 			(effects
@@
 			)
 		)
-		(property "Value" "15p 1%"
+		(property "Value" "15pF 1%"
 			(at 144.78 130.81 90)
 			(effects
@@
 			)
 		)
-		(property "Value" "DMP2037U"
+		(property "Value" "DMP2037U-7"
 			(at 284.48 66.04 90)
 			(effects
@@
 			)
 		)
-		(property "Value" "100p"
+		(property "Value" "100pF"
 			(at 133.35 115.57 0)
 			(effects
@@
 			)
 		)
-		(property "Value" "78n 2% Q=28"
+		(property "Value" "78nH 2% Q=28"
 			(at 139.7 125.222 90)
 			(effects

Commit message: Update all resistors to have an ohm symbol
Make it more clean in the BOM what they are.

Signed-off-by: Corey Minyard <corey@minyard.net>
Parts:
- R52: value 50 -> 50Ω
- R55: value 470 -> 470Ω
Changed lines of the file:
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@@
 			)
 		)
-		(property "Value" "470"
+		(property "Value" "470Ω"
 			(at 255.524 141.986 90)
 			(effects
@@
 			)
 		)
-		(property "Value" "50"
+		(property "Value" "50Ω"
 			(at 178.308 144.653 0)
 			(effects

Commit message: Massive rework of filtering and inductors
Now that I know how inductors really work.

Signed-off-by: Corey Minyard <corey@minyard.net>
Parts:
- L3, L4: value 78nH 2% Q=28 -> 78nH 2%
- L5: value 1nH Q=77 -> 1nH
Other:
- note removed: "See RX1 for Q values on inductors."
Changed lines of the file:
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@@
 		(comment 1 "N5BRG")
-	)
-	(text "See RX1 for Q values on inductors."
-		(exclude_from_sim no)
-		(at 130.302 173.736 0)
-		(effects
-			(font
-				(size 1.524 1.524)
-			)
-			(justify left bottom)
-		)
 	)
 	(text "Rx2+"
@@
 			)
 		)
-		(property "Value" "1nH Q=77"
+		(property "Value" "1nH"
 			(at 171.704 139.446 90)
 			(effects
@@
 			)
 		)
-		(property "Value" "78nH 2% Q=28"
+		(property "Value" "78nH 2%"
 			(at 161.798 139.7 90)
 			(effects
@@
 			)
 		)
-		(property "Value" "78nH 2% Q=28"
+		(property "Value" "78nH 2%"
 			(at 139.7 125.222 90)
 			(effects

Commit message: Have the BOM file fixer output xls, not csv
The omega symbol gets translated properly from xls.

Signed-off-by: Corey Minyard <corey@minyard.net>
Parts:
- FB5: footprint Resistor_SMD:R_0603_1608Metric_Pad0.98x0.95mm_HandSolder -> Inductor_SMD:L_0603_1608Metric_Pad1.05x0.95mm_HandSolder
Changed lines of the file:
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@@
 			)
 		)
-		(property "Footprint" "Resistor_SMD:R_0603_1608Metric_Pad0.98x0.95mm_HandSolder"
+		(property "Footprint" "Inductor_SMD:L_0603_1608Metric_Pad1.05x0.95mm_HandSolder"
 			(at 266.7 71.628 90)
 			(effects

Commit message: Minor fixes for BOM values
Signed-off-by: Corey Minyard <corey@minyard.net>
Parts:
- FB5: value 1K@100MHz -> 1KΩ@100MHz
Changed lines of the file:
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@@
 			)
 		)
-		(property "Value" "1K@100MHz"
+		(property "Value" "1KΩ@100MHz"
 			(at 266.6619 66.04 90)
 			(effects
