File: active_standby.kicad_sch (KiCad schematic)
At the start: 13 parts, among them Q2 BSS138, U24 SN3257QDYYRQ1, U30 SN3257QDYYRQ1

Commit message: Add more infromation about configuration
And add a zero-ohm resistor for bypassing the power off pin.

Signed-off-by: Corey Minyard <corey@minyard.net>
Parts:
- removed R113: 10KΩ, Resistor_SMD:R_0402_1005Metric_Pad0.72x0.64mm_HandSolder, symbol Device:R
- added R118: 0Ω, Resistor_SMD:R_0402_1005Metric_Pad0.72x0.64mm_HandSolder, symbol Device:R
Connections:
- net HW_POWER_OFF1_N: now also R118.1
- net HW_POWER_OFF_N: now also R118.2
Changed lines of the file:
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@@
+	)
+	(junction
+		(at 124.46 140.97)
+		(diameter 0)
+		(color 0 0 0 0)
 	)
 	(junction
@@
 	)
 	(junction
-		(at 63.5 54.61)
+		(at 62.23 151.13)
 		(diameter 0)
 		(color 0 0 0 0)
 	)
 	(junction
-		(at 134.62 140.97)
+		(at 63.5 54.61)
 		(diameter 0)
 		(color 0 0 0 0)
@@
 	(wire
 		(pts
-			(xy 115.57 166.37) (xy 115.57 158.75)
+			(xy 62.23 173.99) (xy 62.23 151.13)
+		)
+		(stroke
+			(width 0)
+			(type default)
+		)
+	)
+	(wire
+		(pts
+			(xy 118.11 180.34) (xy 118.11 158.75)
 		)
 		(stroke
@@
 	(wire
 		(pts
+			(xy 92.71 173.99) (xy 124.46 173.99)
+		)
+		(stroke
+			(width 0)
+			(type default)
+		)
+	)
+	(wire
+		(pts
 			(xy 59.69 35.56) (xy 59.69 41.91)
 		)
@@
 	(wire
 		(pts
-			(xy 134.62 140.97) (xy 143.51 140.97)
+			(xy 124.46 140.97) (xy 143.51 140.97)
 		)
 		(stroke
@@
 	(wire
 		(pts
-			(xy 64.77 156.21) (xy 69.85 156.21)
+			(xy 52.07 156.21) (xy 69.85 156.21)
 		)
 		(stroke
@@
 	(wire
 		(pts
-			(xy 134.62 104.14) (xy 134.62 107.95)
-		)
-		(stroke
-			(width 0)
-			(type default)
-		)
-	)
-	(wire
-		(pts
-			(xy 134.62 115.57) (xy 134.62 140.97)
-		)
-		(stroke
-			(width 0)
-			(type default)
-		)
-	)
-	(wire
-		(pts
 			(xy 52.07 125.73) (xy 62.23 125.73)
 		)
@@
 	(wire
 		(pts
+			(xy 85.09 173.99) (xy 62.23 173.99)
+		)
+		(stroke
+			(width 0)
+			(type default)
+		)
+	)
+	(wire
+		(pts
 			(xy 64.77 148.59) (xy 69.85 148.59)
 		)
@@
 	(wire
 		(pts
-			(xy 110.49 140.97) (xy 134.62 140.97)
+			(xy 110.49 140.97) (xy 124.46 140.97)
 		)
 		(stroke
@@
 	(wire
 		(pts
-			(xy 110.49 158.75) (xy 115.57 158.75)
+			(xy 110.49 158.75) (xy 118.11 158.75)
 		)
 		(stroke
@@
 		(pts
 			(xy 238.76 119.38) (xy 238.76 123.19)
+		)
+		(stroke
+			(width 0)
+			(type default)
+		)
+	)
+	(wire
+		(pts
+			(xy 124.46 173.99) (xy 124.46 140.97)
 		)
 		(stroke
@@
 	(global_label "BOARD_NUM"
 		(shape input)
-		(at 64.77 156.21 180)
+		(at 52.07 156.21 180)
 		(fields_autoplaced yes)
 		(effects
@@
 		)
 		(property "Intersheetrefs" "${INTERSHEET_REFS}"
-			(at 48.4023 156.21 0)
+			(at 35.7023 156.21 0)
 			(effects
 				(font
@@
 				(justify left)
 				(hide yes)
+			)
+		)
+	)
+	(symbol
+		(lib_id "Device:R")
+		(at 88.9 173.99 90)
+		(unit 1)
+		(exclude_from_sim no)
+		(in_bom no)
+		(on_board yes)
+		(dnp yes)
+		(property "Reference" "R118"
+			(at 87.7316 172.212 0)
+			(effects
+				(font
+					(size 1.27 1.27)
+				)
+				(justify left)
+			)
+		)
+		(property "Value" "0Ω"
+			(at 90.043 172.212 0)
+			(effects
+				(font
+					(size 1.27 1.27)
+				)
+				(justify left)
+			)
+		)
+		(property "Footprint" "Resistor_SMD:R_0402_1005Metric_Pad0.72x0.64mm_HandSolder"
+			(at 88.9 175.768 90)
+			(effects
+				(font
+					(size 1.27 1.27)
+				)
+				(hide yes)
+			)
+		)
+		(property "Datasheet" "~"
+			(at 88.9 173.99 0)
+			(effects
+				(font
+					(size 1.27 1.27)
+				)
+				(hide yes)
+			)
+		)
+		(property "Description" ""
+			(at 88.9 173.99 0)
+			(effects
+				(font
+					(size 1.27 1.27)
+				)
+			)
+		)
+		(pin "1"
+		)
+		(pin "2"
+		)
+		(instances
+			(project "PacSat_AFSK"
+				(path "/cc9f42d2-6985-41ac-acab-5ab7b01c5b38/4fa888af-703c-49ed-93bb-d56d2f02c470"
+					(reference "R118")
+					(unit 1)
+				)
 			)
 		)
@@
 	)
 	(symbol
-		(lib_id "power:+3.3V")
-		(at 134.62 104.14 0)
-		(unit 1)
-		(exclude_from_sim no)
-		(in_bom yes)
-		(on_board yes)
-		(dnp no)
-		(fields_autoplaced yes)
-		(property "Reference" "#PWR0268"
-			(at 134.62 107.95 0)
-			(effects
-				(font
-					(size 1.27 1.27)
-				)
-				(hide yes)
-			)
-		)
-		(property "Value" "+3.3V"
-			(at 134.62 100.33 0)
-			(effects
-				(font
-					(size 1.27 1.27)
-				)
-			)
-		)
-		(property "Footprint" ""
-			(at 134.62 104.14 0)
-			(effects
-				(font
-					(size 1.27 1.27)
-				)
-				(hide yes)
-			)
-		)
-		(property "Datasheet" ""
-			(at 134.62 104.14 0)
-			(effects
-				(font
-					(size 1.27 1.27)
-				)
-				(hide yes)
-			)
-		)
-		(property "Description" ""
-			(at 134.62 104.14 0)
-			(effects
-				(font
-					(size 1.27 1.27)
-				)
-			)
-		)
-		(pin "1"
-		)
-		(instances
-			(project "PacSat_AFSK"
-				(path "/cc9f42d2-6985-41ac-acab-5ab7b01c5b38/4fa888af-703c-49ed-93bb-d56d2f02c470"
-					(reference "#PWR0268")
-					(unit 1)
-				)
-			)
-		)
-	)
-	(symbol
 		(lib_id "Transistor_FET:BSS138")
 		(at 133.35 168.91 0)
@@
 		(on_board yes)
 		(dnp no)
-		(fields_autoplaced yes)
 		(property "Reference" "Q2"
-			(at 127 167.6399 0)
+			(at 139.954 162.56 0)
 			(effects
 				(font
@@
 		)
 		(property "Value" "BSS138"
-			(at 127 170.1799 0)
+			(at 139.954 165.1 0)
 			(effects
 				(font
@@
 	(symbol
 		(lib_id "power:GND")
-		(at 115.57 166.37 0)
+		(at 118.11 180.34 0)
 		(unit 1)
 		(exclude_from_sim no)
@@
 		(dnp no)
 		(property "Reference" "#PWR0270"
-			(at 115.57 172.72 0)
+			(at 118.11 186.69 0)
 			(effects
 				(font
@@
 		)
 		(property "Value" "GND"
-			(at 115.697 170.7642 0)
+			(at 118.237 184.7342 0)
 			(effects
 				(font
@@
 		)
 		(property "Footprint" ""
-			(at 115.57 166.37 0)
+			(at 118.11 180.34 0)
 			(effects
 				(font
@@
 		)
 		(property "Datasheet" ""
-			(at 115.57 166.37 0)
+			(at 118.11 180.34 0)
 			(effects
 				(font
@@
 		)
 		(property "Description" ""
-			(at 115.57 166.37 0)
+			(at 118.11 180.34 0)
 			(effects
 				(font
@@
 					(unit 1)
 				)
-			)
-		)
-	)
-	(symbol
-		(lib_id "Device:R")
-		(at 134.62 111.76 0)
-		(unit 1)
-		(exclude_from_sim no)
-		(in_bom yes)
-		(on_board yes)
-		(dnp no)
-		(property "Reference" "R113"
-			(at 136.398 110.5916 0)
-			(effects
-				(font
-					(size 1.27 1.27)
-				)
-				(justify left)
-			)
-		)
-		(property "Value" "10KΩ"
-			(at 136.398 112.903 0)
-			(effects
-				(font
-					(size 1.27 1.27)
-				)
-				(justify left)
-			)
-		)
-		(property "Footprint" "Resistor_SMD:R_0402_1005Metric_Pad0.72x0.64mm_HandSolder"
-			(at 132.842 111.76 90)
-			(effects
-				(font
-					(size 1.27 1.27)
-				)
-				(hide yes)
-			)
-		)
-		(property "Datasheet" "~"
-			(at 134.62 111.76 0)
-			(effects
-				(font
-					(size 1.27 1.27)
-				)
-				(hide yes)
-			)
-		)
-		(property "Description" ""
-			(at 134.62 111.76 0)
-			(effects
-				(font
-					(size 1.27 1.27)
-				)
-			)
-		)
-		(pin "1"
-		)
-		(pin "2"
-		)
-		(instances
-			(project "PacSat_AFSK"
-				(path "/cc9f42d2-6985-41ac-acab-5ab7b01c5b38/4fa888af-703c-49ed-93bb-d56d2f02c470"
-					(reference "R113")
-					(unit 1)
-				)
