File: Clocks.kicad_sch (KiCad schematic)
At the start: 10 parts, among them U3 LMK1C1106A, Y2 O 16,0-JT22CT-A-P-3,3-LF

Commit message: Add a pullup to the LMK1C1106A (clock dist) enable
The spec sheet says to use a pullup, but it was directly connected
to +3.3V.

Signed-off-by: Corey Minyard <corey@minyard.net>
Parts:
- added R114: 10KΩ, Resistor_SMD:R_0402_1005Metric_Pad0.72x0.64mm_HandSolder, symbol Device:R
Connections:
- net at C24.1, C25.1, C26.1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: now also R114.1; no longer U3.2 (1G)
- new net: R114.2, U3.2 (1G)
Changed lines of the file:
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@@
 	(wire
 		(pts
-			(xy 196.85 110.49) (xy 196.85 93.98)
+			(xy 196.85 110.49) (xy 196.85 102.87)
 		)
 		(stroke
@@
 		(pts
 			(xy 213.36 93.98) (xy 215.9 93.98)
+		)
+		(stroke
+			(width 0)
+			(type default)
+		)
+	)
+	(wire
+		(pts
+			(xy 196.85 95.25) (xy 196.85 93.98)
 		)
 		(stroke
@@
 					(unit 1)
 				)
+			)
+		)
+	)
+	(symbol
+		(lib_id "Device:R")
+		(at 196.85 99.06 0)
+		(mirror y)
+		(unit 1)
+		(exclude_from_sim no)
+		(in_bom yes)
+		(on_board yes)
+		(dnp no)
+		(property "Reference" "R114"
+			(at 195.072 97.8916 0)
+			(effects
+				(font
+					(size 1.27 1.27)
+				)
+				(justify left)
+			)
+		)
+		(property "Value" "10KΩ"
+			(at 195.072 100.203 0)
+			(effects
+				(font
+					(size 1.27 1.27)
+				)
+				(justify left)
+			)
+		)
+		(property "Footprint" "Resistor_SMD:R_0402_1005Metric_Pad0.72x0.64mm_HandSolder"
+			(at 198.628 99.06 90)
+			(effects
+				(font
+					(size 1.27 1.27)
+				)
+				(hide yes)
+			)
+		)
+		(property "Datasheet" "~"
+			(at 196.85 99.06 0)
+			(effects
+				(font
+					(size 1.27 1.27)
+				)
+				(hide yes)
+			)
+		)
+		(property "Description" ""
+			(at 196.85 99.06 0)
+			(effects
+				(font
+					(size 1.27 1.27)
+				)
+			)
+		)
+		(pin "1"
+		)
+		(pin "2"
+		)
+		(instances
+			(project "PacSat_AFSK"
+				(path "/cc9f42d2-6985-41ac-acab-5ab7b01c5b38/a735fef7-c3fa-4339-b3a6-fbce810c3c4b"
+					(reference "R114")
+					(unit 1)
+				)
